Commit message: changes made

File: ws_new/install/mobile_robot/share/mobile_robot/model/robot.xacro (robot description, xacro)
@@ -145,5 +145,10 @@
       <parent link="${prefix}_leg"/>
       <child link="${prefix}_wheel"/>
-      <origin xyz="0 0 ${-leg_length_z}" rpy="0 0 ${PI/2}"/>
+      <xacro:if value="${prefix == 'bl'}">
+        <origin xyz="0 0.15 ${-leg_length_z}" rpy="0 0 ${PI/2}"/>
+      </xacro:if>
+      <xacro:if value="${prefix == 'br'}">
+        <origin xyz="0 -0.15 ${-leg_length_z}" rpy="0 0 ${PI/2}"/>
+      </xacro:if>
       <axis xyz="1 0 0"/>
       <dynamics damping="0.01"/>
@@ -213,4 +218,19 @@
     <origin xyz="0 0 0.1" rpy="0 0 0"/>
   </joint>
+  <link name="gps_link">
+    <inertial>
+      <mass>0.1</mass>
+      <inertia>
+        <ixx>0.001</ixx>
+        <iyy>0.001</iyy>
+        <izz>0.001</izz>
+      </inertia>
+    </inertial>
+  </link>
+  <joint name="gps_joint" type="fixed">
+    <parent link="base_link"/>
+    <child link="gps_link"/>
+    <origin xyz="0 0 0.2" rpy="0 0 0"/> <!-- Adjust height as needed -->
+  </joint>
   <!-- Fixed joint connecting the base_link to the body_link -->
   <joint name="body_joint" type="fixed">
@@ -305,8 +325,6 @@
   <!-- This file contains additional Gazebo configurations -->
   <xacro:include filename="$(find mobile_robot)/model/robot.gazebo"/>
-    <!--
-    <xacro:include filename="$(find mobile_robot)/description/"camera.xacro" />
-    <xacro:include filename="$(find mobile_robot)/description/"lidar.xacro" />
-    <xacro:include filename="$(find mobile_robot)/description/"gps.xacro" />
-    -->
+  <!-- <xacro:include filename="$(find mobile_robot)/description/gps.xacro"/> -->
+  <!-- <xacro:include filename="$(find mobile_robot)/description/camera.xacro" />
+  <xacro:include filename="$(find mobile_robot)/description/lidar.xacro" /> -->
 </robot>

Commit message: 30 april

File: ws_new/install/mobile_robot/share/mobile_robot/model/robot.xacro (robot description, xacro)
@@ -216,5 +216,6 @@
     <parent link="base_link"/>
     <child link="imu_link"/>
-    <origin xyz="0 0 0.1" rpy="0 0 0"/>
+    <!-- <origin xyz="0 0 0.1" rpy="0 0 0"/> -->
+    <origin xyz="0 0 0.1" rpy="0 0 0"/> <!--Rotate 180 degrees around x-axis to flip z-axis-->
   </joint>
   <link name="gps_link">
@@ -231,5 +232,5 @@
     <parent link="base_link"/>
     <child link="gps_link"/>
-    <origin xyz="0 0 0.2" rpy="0 0 0"/> <!-- Adjust height as needed -->
+    <origin xyz="0 0 0.2" rpy="0 0 3.14159"/> <!-- Adjust height as needed -->
   </joint>
   <!-- Fixed joint connecting the base_link to the body_link -->

Commit message: 1

File: ws_new/install/mobile_robot/share/mobile_robot/model/robot.xacro (robot description, xacro)
@@ -5,12 +5,14 @@
   <xacro:property name="PI" value="3.1415926535897931"/>
   <!-- Base properties: mass, dimensions -->
-  <xacro:property name="base_mass" value="20.0"/> <!--  CHANGE Body mass (kg) -->
+  <!-- <xacro:property name="base_mass" value="20.0"/>  CHANGE Body mass (kg) -->
+  <xacro:property name="base_mass" value="0.0001"/> <!--  CHANGE Body mass (kg) -->
   <xacro:property name="base_length" value="1.718"/> <!-- Body length (m) -->
   <xacro:property name="base_width" value="1.0"/> <!-- Body width (m) -->
   <xacro:property name="base_height" value="0.3"/> <!-- Body height (m) -->
   <!-- Wheelbase is the distance between the front and rear axles -->
-  <xacro:property name="wheelbase" value="1.08"/> <!-- Distance between front and rear axles (m) -->
+  <xacro:property name="wheelbase" value="1.364"/> <!-- Distance between front and rear axles (m) -->
   <!-- Wheel properties -->
-  <xacro:property name="wheel_mass" value="1.0"/> <!-- Wheel mass (kg) -->
+  <!-- <xacro:property name="wheel_mass" value="1.0"/> Wheel mass (kg) -->
+  <xacro:property name="wheel_mass" value="0.0001"/>
   <xacro:property name="wheel_len" value="0.241"/> <!-- Wheel width (m) -->
   <xacro:property name="wheel_radius" value="0.235"/> <!-- Wheel radius (m) -->
@@ -20,5 +22,6 @@
   <xacro:property name="leg_length_z" value="0.530"/>
   <xacro:property name="leg_angle" value="${radians(15)}"/> <!-- Leg tilt angle -->
-  <xacro:property name="leg_mass" value="10.0"/> <!-- Leg mass (kg) -->
+  <!-- <xacro:property name="leg_mass" value="10.0"/> Leg mass (kg) -->
+  <xacro:property name="leg_mass" value="0.00001"/>
   <!-- Macro for Legs with Wheels -->
   <!-- This macro instantiates a leg and its attached wheel. Parameters:
