Commit message: 1

File: ws_new/install/mobile_robot/share/mobile_robot/description/camera.xacro (robot description, xacro)
@@ -1 +1,52 @@
-/home/thomas/MobileRobot/ws_new/src/mobile_robot/description/camera.xacro
+<?xml version="1.0"?>
+<robot xmlns:xacro="http://www.ros.org/wiki/xacro" >
+    <joint name="camera_joint" type="fixed">
+        <parent link="chassis"/>
+        <child link="camera_link"/>
+        <origin xyz="1.718 0 0.181" rpy="0 0 0"/>
+    </joint>
+    <link name="camera_link">
+        <visual>
+            <geometry>
+                <box size="0.010 0.03 0.03"/>
+            </geometry>
+            <material name="black"/>
+        </visual>
+        <visual>
+            <origin xyz="0 0 -0.05"/>
+            <geometry>
+                <cylinder radius="0.002" length="0.1"/>
+            </geometry>
+            <material name="black"/>
+        </visual>
+    </link>
+    <joint name="camera_optical_joint" type="fixed">
+        <parent link="camera_link"/>
+        <child link="camera_link_optical"/>
+        <origin xyz="0 0 0" rpy="${-pi/2} 0 ${-pi/2}"/>
+    </joint>
+    <link name="camera_link_optical"></link>
+    <gazebo reference="camera_link">
+        <material>Gazebo/Black</material>
+        <sensor name="camera" type="camera">
+            <pose> 0 0 0 0 0 0 </pose>
+            <visualize>true</visualize>
+            <update_rate>10</update_rate>
+            <camera>
+                <camera_info_topic>camera/camera_info</camera_info_topic>
+                <horizontal_fov>1.089</horizontal_fov>
+                <image>
+                    <format>R8G8B8</format>
+                    <width>640</width>
+                    <height>480</height>
+                </image>
+                <clip>
+                    <near>0.05</near>
+                    <far>8.0</far>
+                </clip>
+            </camera>
+            <topic>camera/image_raw</topic>
+            <gz_frame_id>camera_link_optical</gz_frame_id>
+        </sensor>
+    </gazebo>
+</robot>

File: ws_new/install/mobile_robot/share/mobile_robot/description/lidar.xacro (robot description, xacro)
@@ -1 +1,54 @@
-/home/thomas/MobileRobot/ws_new/src/mobile_robot/description/lidar.xacro
+<?xml version="1.0"?>
+<robot xmlns:xacro="http://www.ros.org/wiki/xacro" >
+    <link name="laser_frame">
+        <visual>
+            <geometry>
+                <cylinder radius="0.05" length="0.04"/>
+            </geometry>
+            <material name="black"/>
+        </visual>
+        <visual>
+            <origin xyz="0 0 -0.05"/>
+            <geometry>
+                <cylinder radius="0.01" length="0.1"/>
+            </geometry>
+            <material name="black"/>
+        </visual>
+        <collision>
+            <geometry>
+                <cylinder radius="0.05" length="0.04"/>
+            </geometry>
+        </collision>
+        <xacro:inertial_cylinder mass="0.1" length="0.04" radius="0.05">
+            <origin xyz="0 0 0" rpy="0 0 0"/>
+        </xacro:inertial_cylinder>
+    </link>
+    <joint name="laser_joint" type="fixed">
+        <parent link="body_link"/>
+        <child link="laser_frame"/>
+        <origin xyz="0.122 0 0.212" rpy="0 0 0"/>
+    </joint>
+    <gazebo reference="laser_frame">
+        <material>Gazebo/Black</material>
+        <sensor name="laser" type="gpu_lidar">
+            <pose> 0 0 0 0 0 0 </pose>
+            <visualize>false</visualize>
+            <update_rate>10</update_rate>
+            <lidar>
+                <scan>
+                    <horizontal>
+                        <samples>360</samples>
+                        <min_angle>-3.14</min_angle>
+                        <max_angle>3.14</max_angle>
+                    </horizontal>
+                </scan>
+                <range>
+                    <min>0.3</min>
+                    <max>12</max>
+                </range>
+            </lidar>
+            <topic>scan</topic>
+            <gz_frame_id>laser_frame</gz_frame_id>
+        </sensor>
+    </gazebo>
+</robot>

File: ws_new/install/mobile_robot/share/mobile_robot/model/robot.xacro (robot description, xacro)
@@ -1 +1,364 @@
-/home/thomas/MobileRobot/ws_new/src/mobile_robot/model/robot.xacro
+<?xml version="1.0"?>
+<robot name="ackerman_drive_robot" xmlns:xacro="http://www.ros.org/wiki/xacro">
+  <!-- Properties -->
+  <!-- Define constant PI -->
+  <xacro:property name="PI" value="3.1415926535897931"/>
+  <!-- Base properties: mass, dimensions -->
+  <!-- <xacro:property name="base_mass" value="20.0"/>  CHANGE Body mass (kg) -->
+  <xacro:property name="base_mass" value="0.0001"/> <!--  CHANGE Body mass (kg) -->
+  <xacro:property name="base_length" value="1.718"/> <!-- Body length (m) -->
+  <xacro:property name="base_width" value="1.0"/> <!-- Body width (m) -->
+  <xacro:property name="base_height" value="0.3"/> <!-- Body height (m) -->
+  <!-- Wheelbase is the distance between the front and rear axles -->
+  <xacro:property name="wheelbase" value="1.364"/> <!-- Distance between front and rear axles (m) -->
+  <!-- Wheel properties -->
+  <!-- <xacro:property name="wheel_mass" value="1.0"/> Wheel mass (kg) -->
+  <xacro:property name="wheel_mass" value="0.0001"/>
+  <xacro:property name="wheel_len" value="0.241"/> <!-- Wheel width (m) -->
+  <xacro:property name="wheel_radius" value="0.235"/> <!-- Wheel radius (m) -->
+  <!-- Leg properties -->
+  <xacro:property name="leg_length_x" value="0.06"/> <!-- Leg dimensions (m) -->
+  <xacro:property name="leg_length_y" value="0.040"/>
+  <xacro:property name="leg_length_z" value="0.530"/>
+  <xacro:property name="leg_angle" value="${radians(15)}"/> <!-- Leg tilt angle -->
+  <!-- <xacro:property name="leg_mass" value="10.0"/> Leg mass (kg) -->
+  <xacro:property name="leg_mass" value="0.00001"/>
+  <!-- Macro for Legs with Wheels -->
+  <!-- This macro instantiates a leg and its attached wheel. Parameters:
+         prefix: used to name the leg and wheel uniquely,
+         leg_origin_xyz: position of the leg joint,
+         leg_origin_rpy: orientation of the leg joint,
+         wheel_joint_type: the type of joint for the wheel (revolute or continuous) -->
+  <xacro:macro name="leg_with_wheel" params="prefix leg_origin_xyz leg_origin_rpy wheel_joint_type is_front_wheel">
+    <!-- Leg Link -->
+    <link name="${prefix}_leg">
+      <inertial>
+        <origin xyz="0 0 ${-leg_length_z/2}" rpy="0 0 0"/>
+        <mass value="${leg_mass}"/>
+        <inertia
+          ixx="${(1/12)*leg_mass*(leg_length_y*leg_length_y + leg_length_z*leg_length_z)}"
+          ixy="0.0" ixz="0.0"
+          iyy="${(1/12)*leg_mass*(leg_length_x*leg_length_x + leg_length_z*leg_length_z)}"
+          iyz="0.0"
+          izz="${(1/12)*leg_mass*(leg_length_x*leg_length_x + leg_length_y*leg_length_y)}"/>
+      </inertial>
+      <visual>
+        <origin xyz="0 0 ${-leg_length_z/2}" rpy="0 0 0"/>
+        <geometry>
+          <box size="${leg_length_x} ${leg_length_y} ${leg_length_z}"/>
+        </geometry>
+        <material name="gray">
+          <color rgba="0.5 0.5 0.5 1"/> <!-- Gray for visibility -->
+        </material>
+      </visual>
+      <collision>
+        <origin xyz="0 0 ${-leg_length_z/2}" rpy="0 0 0"/>
+        <geometry>
+          <box size="${leg_length_x} ${leg_length_y} ${leg_length_z}"/>
+        </geometry>
+      </collision>
+    </link>
+    <!-- Fixed joint to attach the leg to the body link -->
+    <joint name="${prefix}_leg_joint" type="fixed">
+      <parent link="body_link"/>
+      <child link="${prefix}_leg"/>
+      <origin xyz="${leg_origin_xyz}" rpy="${leg_origin_rpy}"/>
+    </joint>
+    <!-- Wheel Link -->
+    <link name="${prefix}_wheel">
+      <inertial>
+        <!-- Wheel inertial parameters: rotated so that cylinder axis is along the proper direction -->
+        <origin xyz="0 0 0" rpy="${PI/2} 0 ${PI/2}"/>
+        <mass value="${wheel_mass}"/>
+        <inertia
+          ixx="${(1/12)*wheel_mass*(3*wheel_radius*wheel_radius + wheel_len*wheel_len)}"
+          ixy="0.0" ixz="0.0"
+          iyy="${(1/12)*wheel_mass*(3*wheel_radius*wheel_radius + wheel_len*wheel_len)}"
+          iyz="0.0"
+          izz="${(1/2)*wheel_mass*wheel_radius*wheel_radius}"/>
+      </inertial>
+      <visual>
+        <origin xyz="0 0 0" rpy="${PI/2} 0 ${PI/2}"/>
+        <geometry>
+          <cylinder length="${wheel_len}" radius="${wheel_radius}"/>
+        </geometry>
+        <material name="black">
+          <color rgba="0 0 0 1"/> <!-- Black for visibility -->
+        </material>
+      </visual>
+      <collision>
+        <origin xyz="0 0 0" rpy="${PI/2} 0 ${PI/2} "/>
+        <geometry>
+          <cylinder length="${wheel_len}" radius="${wheel_radius}"/>
+        </geometry>
+      </collision>
+    </link>
+    <xacro:if value="${is_front_wheel}">
+    <link name="${prefix}_steering_link">
+      <!-- Inertial properties: Minimal mass and inertia since this is a lightweight steering component. -->
+      <inertial>
+        <mass value="0.1"/>
+        <!-- Simple inertia values (small, uniform) for simulation stability. -->
+        <inertia ixx="0.001" ixy="0.0" ixz="0.0" iyy="0.001" iyz="0.0" izz="0.001"/>
+      </inertial>
+      <visual>
+        <origin xyz="0 0 0" rpy="${PI/2} 0 ${PI/2}"/>
+        <geometry>
+          <cylinder length="0.01" radius="0.01"/>
+        </geometry>
+        <material name="invisible"/>
+      </visual>
+    </link>
+      <!-- FRONT WHEELS-->
+      <!-- Steering Joint: Allows the steering link to rotate (steer) around the vertical axis. -->
+      <joint name="${prefix}_steering_joint" type="revolute">
+        <parent link="${prefix}_leg"/> <!-- Parent is the leg link. -->
+        <child link="${prefix}_steering_link"/>  <!-- Child is the steering link. -->
+        <origin xyz="0 0 ${-leg_length_z}" rpy="0 ${leg_angle} 0"/> <!-- Positioned at the bottom of the leg (z offset). -->
+        <axis xyz="0 0 1"/> <!-- Rotation axis is vertical (z-axis) for steering left/right. -->
+        <!-- Limits: Steering angle range. effort, and velocity constraints. -->
+        <limit lower="-0.4" upper="0.4" effort="100000.0" velocity="10.0"/>
+        <dynamics damping="0.2"/>
+      </joint>
+      <!-- Joint connecting steering and the wheel -->
+      <joint name="${prefix}_wheel_joint" type="${wheel_joint_type}">
+        <parent link="${prefix}_steering_link"/>
+        <child link="${prefix}_wheel"/>
+        <!-- Conditionally set the lateral offset:
+            For the left wheel (prefix "fl"), offset +0.15 in y;
+            For the right wheel (prefix "fr"), offset -0.15 in y.
+            Adjust the third value (-0.1) as needed for the z offset. -->
+        <xacro:if value="${prefix == 'fl'}">
+          <origin xyz="0 0.15 -0.0" rpy="0 0 ${PI/2}"/>  <!-- WRONG   ${-leg_angle} -->
+        </xacro:if>
+        <xacro:if value="${prefix == 'fr'}">
+          <origin xyz="0 -0.15 -0.0" rpy="0 0 ${PI/2}"/> <!-- WRONG   ${-leg_angle}-->
+        </xacro:if>
+        <axis xyz="1 0 0"/>
+        <dynamics damping="0.2"/>
+        <!-- Apply limits only if the joint is revolute -->
+        <xacro:if value="${wheel_joint_type == 'revolute'}">
+          <limit lower="-0.5" upper="0.5" effort="100.0" velocity="10.0"/>
+        </xacro:if>
+      </joint>
+    </xacro:if>
+    <!-- Back Wheels: No steering; wheel is directly attached to the leg. -->
+  <xacro:unless value="${is_front_wheel}">
+    <joint name="${prefix}_wheel_joint" type="${wheel_joint_type}">
+      <parent link="${prefix}_leg"/>
+      <child link="${prefix}_wheel"/>
+      <xacro:if value="${prefix == 'bl'}">
+        <origin xyz="0 0.15 ${-leg_length_z}" rpy="0 0 ${PI/2}"/>
+      </xacro:if>
+      <xacro:if value="${prefix == 'br'}">
+        <origin xyz="0 -0.15 ${-leg_length_z}" rpy="0 0 ${PI/2}"/>
+      </xacro:if>
+      <axis xyz="1 0 0"/>
+      <dynamics damping="0.01"/>
+      <!-- If the joint is revolute, then apply limits -->
+      <xacro:if value="${wheel_joint_type == 'revolute'}">
+      </xacro:if>
+    </joint>
+  </xacro:unless>
+  </xacro:macro>
+  <!-- Base Link (World Reference) -->
+  <!-- The base_link serves as the fixed reference frame for the robot model -->
+  <link name="base_link"/>
+  <!-- BASE_FOOTPRINT LINK -->
+  <joint name="base_footprint_joint" type="fixed">
+      <parent link="base_link"/>
+      <child link="base_footprint"/>
+      <origin xyz="0 0 0" rpy="0 0 0"/>
+  </joint>
+  <link name="base_footprint">
+  </link>
+  <!-- Body Link -->
+  <link name="body_link">
+    <inertial>
+      <origin xyz="0 0 0" rpy="0 0 0"/>
+      <mass value="${base_mass}"/>
+      <inertia
+        ixx="${(1/12)*base_mass*(base_width*base_width + base_height*base_height)}"
+        ixy="0.0" ixz="0.0"
+        iyy="${(1/12)*base_mass*(base_length*base_length + base_height*base_height)}"
+        iyz="0.0"
+        izz="${(1/12)*base_mass*(base_length*base_length + base_width*base_width)}"/>
+    </inertial>
+    <visual>
+      <origin xyz="0 0 0" rpy="0 0 0"/>
+      <geometry>
+        <box size="${base_length} ${base_width} ${base_height}"/>
+      </geometry>
+      <material name="blue">
+        <color rgba="0 0 1 1"/> <!-- Blue for visibility -->
+      </material>
+    </visual>
+    <collision>
+      <origin xyz="0 0 0" rpy="0 0 0"/>
+      <geometry>
+        <box size="${base_length} ${base_width} ${base_height}"/>
+      </geometry>
+    </collision>
+  </link>
+ <!-- imu -->
+  <link name="imu_link">
+    <inertial>
+      <mass value="0.1"/>
+      <inertia ixx="0.001" ixy="0.0" ixz="0.0" iyy="0.001" iyz="0.0" izz="0.001"/>
+    </inertial>
+    <visual>
+      <geometry>
+        <box size="0.02 0.02 0.02"/>
+      </geometry>
+      <material name="white">
+        <color rgba="1 1 1 1"/>
+      </material>
+    </visual>
+  </link>
+  <joint name="imu_joint" type="fixed">
+    <parent link="base_link"/>
+    <child link="imu_link"/>
+    <!-- <origin xyz="0 0 0.1" rpy="0 0 0"/> -->
+    <origin xyz="0 0 0.1" rpy="0 0 0"/> <!--Rotate 180 degrees around x-axis to flip z-axis-->
+  </joint>
+  <link name="gps_link">
+    <inertial>
+      <mass>0.1</mass>
+      <inertia>
+        <ixx>0.001</ixx>
+        <iyy>0.001</iyy>
+        <izz>0.001</izz>
+      </inertia>
+    </inertial>
+  </link>
+  <joint name="gps_joint" type="fixed">
+    <parent link="base_link"/>
+    <child link="gps_link"/>
+    <origin xyz="0 0 0.2" rpy="0 0 3.14159"/> <!-- Adjust height as needed -->
+  </joint>
+  <!-- Fixed joint connecting the base_link to the body_link -->
+  <joint name="body_joint" type="fixed">
+    <parent link="base_link"/>
+    <child link="body_link"/>
+    <origin xyz="0 0 ${base_height/2 + leg_length_z + wheel_radius}" rpy="0 0 0"/>
+  </joint>
+  <!-- Instantiate Legs with Wheels -->
+  <!-- Front Left Leg with Wheel -->
+  <xacro:leg_with_wheel prefix="fl" leg_origin_xyz="${wheelbase/2} ${base_width/2} ${-base_height/2}" leg_origin_rpy="0 ${-leg_angle} 0" wheel_joint_type="continuous" is_front_wheel="true"/>
+  <!-- Front Right Leg with Wheel -->
+  <xacro:leg_with_wheel prefix="fr" leg_origin_xyz="${wheelbase/2} ${-base_width/2} ${-base_height/2}" leg_origin_rpy="0 ${-leg_angle} 0" wheel_joint_type="continuous" is_front_wheel="true"/>
+  <!-- Back Left Leg with Wheel -->
+  <xacro:leg_with_wheel prefix="bl" leg_origin_xyz="${-wheelbase/2} ${base_width/2} ${-base_height/2}" leg_origin_rpy="0 ${leg_angle} 0" wheel_joint_type="continuous" is_front_wheel="false"/>
+  <!-- Back Right Leg with Wheel -->
+  <xacro:leg_with_wheel prefix="br" leg_origin_xyz="${-wheelbase/2} ${-base_width/2} ${-base_height/2}" leg_origin_rpy="0 ${leg_angle} 0" wheel_joint_type="continuous" is_front_wheel="false"/>
+  <!-- LIDAR -->
+  <link name="laser_frame">
+      <visual>
+          <geometry>
+              <cylinder radius="0.05" length="0.04"/>
+          </geometry>
+          <material name="black"/>
+      </visual>
+      <visual>
+          <origin xyz="0 0 -0.05"/>
+          <geometry>
+              <cylinder radius="0.01" length="0.1"/>
+          </geometry>
+          <material name="black"/>
+      </visual>
+      <collision>
+          <geometry>
+              <cylinder radius="0.05" length="0.04"/>
+          </geometry>
+      </collision>
+      <!-- Explicit inertial definition -->
+      <inertial>
+          <mass value="0.1"/>
+          <inertia ixx="0.0" ixy="0.0" ixz="0.0" iyy="0.0" iyz="0.0" izz="0.0"/>
+      </inertial>
+      <origin xyz="0 0 0" rpy="0 0 0"/>
+  </link>
+  <joint name="laser_joint" type="fixed">
+      <parent link="body_link"/>
+      <child link="laser_frame"/>
+      <origin xyz="0.122 0 0.212" rpy="0 0 0"/>
+  </joint>
+  <ros2_control name="GazeboSystem" type="system">
+    <hardware>
+        <plugin>gz_ros2_control/GazeboSimSystem</plugin>
+    </hardware>
+    <joint name="fl_steering_joint">
+      <command_interface name="position"/>
+      <state_interface name="position"/>
+      <state_interface name="velocity"/>
+    </joint>
+    <joint name="fr_steering_joint">
+      <command_interface name="position"/>
+      <state_interface name="position"/>
+      <state_interface name="velocity"/>
+    </joint>
+    <joint name="bl_wheel_joint">
+      <command_interface name="velocity"/>
+      <state_interface name="position"/>
+      <state_interface name="velocity"/>
+    </joint>
+    <joint name="br_wheel_joint">
+      <command_interface name="velocity"/>
+      <state_interface name="position"/>
+      <state_interface name="velocity"/>
+    </joint>
+    <!--To show them in rviz  -->
+    <joint name="fl_wheel_joint">
+      <command_interface name="velocity"/>
+      <state_interface name="position"/>
+      <state_interface name="velocity"/>
+    </joint>
+    <joint name="fr_wheel_joint">
+      <command_interface name="velocity"/>
+      <state_interface name="position"/>
+      <state_interface name="velocity"/>
+    </joint>
+  </ros2_control>
+  <!-- Transmission Elements -->
+  <!-- Transmissions map joint commands to actuator commands -->
+  <!--
+  This defines a transmission between an actuator and a joint.
+  - 'SimpleTransmission' assumes a 1:1 mapping (no reduction or gearing).
+  - The actuator (fl_wheel_actuator) will control the joint (fl_wheel_joint).
+  - Required by ros2_control to map control commands to physical or simulated hardware.
+-->
+  <transmission name="fl_steering_trans">
+    <type>transmission_interface/SimpleTransmission</type>
+    <joint name="fl_steering_joint"/>
+    <actuator name="fl_steering_actuator"/>
+  </transmission>
+  <transmission name="fr_steering_trans">
+    <type>transmission_interface/SimpleTransmission</type>
+    <joint name="fr_steering_joint"/>
+    <actuator name="fr_steering_actuator"/>
+  </transmission>
+  <transmission name="bl_wheel_trans">
+    <type>transmission_interface/SimpleTransmission</type>
+    <joint name="bl_wheel_joint"/>
+    <actuator name="bl_wheel_actuator"/>
+  </transmission>
+  <transmission name="br_wheel_trans">
+    <type>transmission_interface/SimpleTransmission</type>
+    <joint name="br_wheel_joint"/>
+    <actuator name="br_wheel_actuator"/>
+  </transmission>
+  <transmission name="fl_wheel_trans">
+    <type>transmission_interface/SimpleTransmission</type>
+    <joint name="fl_wheel_joint"/>
+    <actuator name="fl_wheel_actuator"/>
+  </transmission>
+  <transmission name="fr_wheel_trans">
+    <type>transmission_interface/SimpleTransmission</type>
+    <joint name="fr_wheel_joint"/>
+    <actuator name="fr_wheel_actuator"/>
+  </transmission>
+  <!-- Include Gazebo-specific file -->
+  <!-- This file contains additional Gazebo configurations -->
+  <xacro:include filename="$(find mobile_robot)/model/robot.gazebo"/>
+  <!-- <xacro:include filename="$(find mobile_robot)/description/camera.xacro" /> -->
+</robot>
